Commit message: add

File: cartesian_controller_simulation/urdf/ur5.urdf (robot description, URDF)
Before this commit: robot ur5, 9 links, 8 joints
Links:
- link base_link: geometry collision mesh filename=file:///home/parallels/ros2_ws/src/cartesian_controllers/ca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; visual mesh filename=file:///home/parallels/ros2_ws/src/cartesian_controllers/ca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
- link forearm_link: geometry collision mesh filename=file:///home/parallels/ros2_ws/src/cartesian_controllers/ca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; visual mesh filename=file:///home/parallels/ros2_ws/src/cartesian_controllers/ca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
- link shoulder_link: geometry collision mesh filename=file:///home/parallels/ros2_ws/src/cartesian_controllers/ca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; visual mesh filename=file:///home/parallels/ros2_ws/src/cartesian_controllers/ca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
- link upper_arm_link: geometry collision mesh filename=file:///home/parallels/ros2_ws/src/cartesian_controllers/ca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; visual mesh filename=file:///home/parallels/ros2_ws/src/cartesian_controllers/ca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
- link wrist_1_link: geometry collision mesh filename=file:///home/parallels/ros2_ws/src/cartesian_controllers/ca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; visual mesh filename=file:///home/parallels/ros2_ws/src/cartesian_controllers/ca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
- link wrist_2_link: geometry collision mesh filename=file:///home/parallels/ros2_ws/src/cartesian_controllers/ca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; visual mesh filename=file:///home/parallels/ros2_ws/src/cartesian_controllers/ca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
- link wrist_3_link: geometry collision mesh filename=file:///home/parallels/ros2_ws/src/cartesian_controllers/ca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; visual mesh filename=file:///home/parallels/ros2_ws/src/cartesian_controllers/ca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

File: cartesian_controller_simulation/urdf/ur5.urdf.xacro (robot description, xacro)
@@ -3,19 +3,5 @@
   <xacro:include filename="$(find cartesian_controller_simulation)/urdf/ur5.transmission.xacro" />
   <xacro:include filename="$(find cartesian_controller_simulation)/urdf/ur5.gazebo.xacro" />
-  <xacro:include filename="$(find cartesian_controller_simulation)/urdf/joint.urdf.xacro"/>
-  <!-- <xacro:property name="pi" value="3.14159265" /> -->
-        <!-- ROS2 control interfaces -->
-        <ros2_control name="cartesian_controller_simulation" type="system">
-                <xacro:joint_interface name="joint1" p="1000" d="0.5" />
-                <xacro:joint_interface name="joint2" p="1000" d="0.5" />
-                <xacro:joint_interface name="joint3" p="500" d="0.5" />
-                <xacro:joint_interface name="joint4" p="100" d="0.5" />
-                <xacro:joint_interface name="joint5" p="10" d="0.5" />
-                <xacro:joint_interface name="joint6" p="10" d="0.5" />
-                <hardware>
-                        <plugin>cartesian_controller_simulation/Simulator</plugin>
-                        <param name="mujoco_model">$(arg mujoco_model)</param>
-                </hardware>
-        </ros2_control>
+  <!--<xacro:property name="pi" value="3.14159265" />-->
   <!-- Inertia parameters -->
   <xacro:property name="base_mass" value="4.0" />  <!-- This mass might be incorrect -->
