Commit message: add

File: cartesian_controller_simulation/urdf/ur5.urdf.xacro (robot description, xacro)
@@ -1,6 +1,6 @@
 <?xml version="1.0"?>
 <robot name="ur5" xmlns:xacro="http://www.ros.org/wiki/xacro">
-  <xacro:include filename="$(find cartesian_controller_simulation)/urdf/ur5.transmission.xacro" />
-  <xacro:include filename="$(find cartesian_controller_simulation)/urdf/ur5.gazebo.xacro" />
+  <xacro:include filename="/home/parallels/ros2_ws/src/cartesian_controllers/cartesian_controller_simulation/urdf/ur5.transmission.xacro" />
+  <xacro:include filename="/home/parallels/ros2_ws/src/cartesian_controllers/cartesian_controller_simulation/urdf/ur5.gazebo.xacro" />
   <!--<xacro:property name="pi" value="3.14159265" />-->
   <!-- Inertia parameters -->
@@ -72,13 +72,13 @@
       <visual>
         <geometry>
-          <mesh filename="file://$(find cartesian_controller_simulation)/meshes/ur5/visual/Base.dae" />
-        </geometry>
-        <material name="LightGrey">
-          <color rgba="0.7 0.7 0.7 1.0"/>
-        </material>
-      </visual>
-      <collision>
-        <geometry>
-          <mesh filename="file://$(find cartesian_controller_simulation)/meshes/ur5/collision/base.stl" />
+          <mesh filename="file:///home/parallels/ros2_ws/src/cartesian_controllers/cartesian_controller_simulation/meshes/ur5/visual/Base.dae" />
+        </geometry>
+        <material name="LightGrey">
+          <color rgba="0.7 0.7 0.7 1.0"/>
+        </material>
+      </visual>
+      <collision>
+        <geometry>
+          <mesh filename="file:///home/parallels/ros2_ws/src/cartesian_controllers/cartesian_controller_simulation/meshes/ur5/collision/base.stl" />
         </geometry>
       </collision>
@@ -103,13 +103,13 @@
       <visual>
         <geometry>
-          <mesh filename="file://$(find cartesian_controller_simulation)/meshes/ur5/visual/Shoulder.dae" />
-        </geometry>
-        <material name="LightGrey">
-          <color rgba="0.7 0.7 0.7 1.0"/>
-        </material>
-      </visual>
-      <collision>
-        <geometry>
-          <mesh filename="file://$(find cartesian_controller_simulation)/meshes/ur5/collision/shoulder.stl" />
+          <mesh filename="file:///home/parallels/ros2_ws/src/cartesian_controllers/cartesian_controller_simulation/meshes/ur5/visual/Shoulder.dae" />
+        </geometry>
+        <material name="LightGrey">
+          <color rgba="0.7 0.7 0.7 1.0"/>
+        </material>
+      </visual>
+      <collision>
+        <geometry>
+          <mesh filename="file:///home/parallels/ros2_ws/src/cartesian_controllers/cartesian_controller_simulation/meshes/ur5/collision/shoulder.stl" />
         </geometry>
       </collision>
@@ -134,13 +134,13 @@
       <visual>
         <geometry>
-          <mesh filename="file://$(find cartesian_controller_simulation)/meshes/ur5/visual/UpperArm.dae" />
-        </geometry>
-        <material name="LightGrey">
-          <color rgba="0.7 0.7 0.7 1.0"/>
-        </material>
-      </visual>
-      <collision>
-        <geometry>
-          <mesh filename="file://$(find cartesian_controller_simulation)/meshes/ur5/collision/upper_arm.stl" />
+          <mesh filename="file:///home/parallels/ros2_ws/src/cartesian_controllers/cartesian_controller_simulation/meshes/ur5/visual/UpperArm.dae" />
+        </geometry>
+        <material name="LightGrey">
+          <color rgba="0.7 0.7 0.7 1.0"/>
+        </material>
+      </visual>
+      <collision>
+        <geometry>
+          <mesh filename="file:///home/parallels/ros2_ws/src/cartesian_controllers/cartesian_controller_simulation/meshes/ur5/collision/upper_arm.stl" />
         </geometry>
       </collision>
@@ -165,13 +165,13 @@
       <visual>
         <geometry>
-          <mesh filename="file://$(find cartesian_controller_simulation)/meshes/ur5/visual/Forearm.dae" />
-        </geometry>
-        <material name="LightGrey">
-          <color rgba="0.7 0.7 0.7 1.0"/>
-        </material>
-      </visual>
-      <collision>
-        <geometry>
-          <mesh filename="file://$(find cartesian_controller_simulation)/meshes/ur5/collision/forearm.stl" />
+          <mesh filename="file:///home/parallels/ros2_ws/src/cartesian_controllers/cartesian_controller_simulation/meshes/ur5/visual/Forearm.dae" />
+        </geometry>
+        <material name="LightGrey">
+          <color rgba="0.7 0.7 0.7 1.0"/>
+        </material>
+      </visual>
+      <collision>
+        <geometry>
+          <mesh filename="file:///home/parallels/ros2_ws/src/cartesian_controllers/cartesian_controller_simulation/meshes/ur5/collision/forearm.stl" />
         </geometry>
       </collision>
@@ -196,13 +196,13 @@
       <visual>
         <geometry>
-          <mesh filename="file://$(find cartesian_controller_simulation)/meshes/ur5/visual/Wrist1.dae" />
-        </geometry>
-        <material name="LightGrey">
-          <color rgba="0.7 0.7 0.7 1.0"/>
-        </material>
-      </visual>
-      <collision>
-        <geometry>
-          <mesh filename="file://$(find cartesian_controller_simulation)/meshes/ur5/collision/wrist_1.stl" />
+          <mesh filename="file:///home/parallels/ros2_ws/src/cartesian_controllers/cartesian_controller_simulation/meshes/ur5/visual/Wrist1.dae" />
+        </geometry>
+        <material name="LightGrey">
+          <color rgba="0.7 0.7 0.7 1.0"/>
+        </material>
+      </visual>
+      <collision>
+        <geometry>
+          <mesh filename="file:///home/parallels/ros2_ws/src/cartesian_controllers/cartesian_controller_simulation/meshes/ur5/collision/wrist_1.stl" />
         </geometry>
       </collision>
@@ -227,13 +227,13 @@
       <visual>
         <geometry>
-          <mesh filename="file://$(find cartesian_controller_simulation)/meshes/ur5/visual/Wrist2.dae" />
-        </geometry>
-        <material name="LightGrey">
-          <color rgba="0.7 0.7 0.7 1.0"/>
-        </material>
-      </visual>
-      <collision>
-        <geometry>
-          <mesh filename="file://$(find cartesian_controller_simulation)/meshes/ur5/collision/wrist_2.stl" />
+          <mesh filename="file:///home/parallels/ros2_ws/src/cartesian_controllers/cartesian_controller_simulation/meshes/ur5/visual/Wrist2.dae" />
+        </geometry>
+        <material name="LightGrey">
+          <color rgba="0.7 0.7 0.7 1.0"/>
+        </material>
+      </visual>
+      <collision>
+        <geometry>
+          <mesh filename="file:///home/parallels/ros2_ws/src/cartesian_controllers/cartesian_controller_simulation/meshes/ur5/collision/wrist_2.stl" />
         </geometry>
       </collision>
@@ -258,13 +258,13 @@
       <visual>
         <geometry>
-          <mesh filename="file://$(find cartesian_controller_simulation)/meshes/ur5/visual/Wrist3.dae" />
-        </geometry>
-        <material name="LightGrey">
-          <color rgba="0.7 0.7 0.7 1.0"/>
-        </material>
-      </visual>
-      <collision>
-        <geometry>
-          <mesh filename="file://$(find cartesian_controller_simulation)/meshes/ur5/collision/wrist_3.stl" />
+          <mesh filename="file:///home/parallels/ros2_ws/src/cartesian_controllers/cartesian_controller_simulation/meshes/ur5/visual/Wrist3.dae" />
+        </geometry>
+        <material name="LightGrey">
+          <color rgba="0.7 0.7 0.7 1.0"/>
+        </material>
+      </visual>
+      <collision>
+        <geometry>
+          <mesh filename="file:///home/parallels/ros2_ws/src/cartesian_controllers/cartesian_controller_simulation/meshes/ur5/collision/wrist_3.stl" />
         </geometry>
       </collision>
